Commit message: Making emma model

File: src/emma_visualization/description/emma.urdf.xacro (robot description, xacro)
@@ -1,5 +1,4 @@
 <?xml version="1.0"?>
 <robot xmlns:xacro="http://www.ros.org/wiki/xacro" name="emma_robot">
-    <!--Example Link-->
-    <link name="base_link"></link>
+    <xacro:include filename="emma_core.xacro" />
 </robot>

Commit message: using stl as visual only without collision enabled for testing

File: src/emma_visualization/description/emma.urdf.xacro (robot description, xacro)
@@ -2,3 +2,4 @@
 <robot xmlns:xacro="http://www.ros.org/wiki/xacro" name="emma_robot">
     <xacro:include filename="emma_core.xacro" />
+    <xacro:include filename="gazebo_control.xacro" />
 </robot>

File: src/emma_visualization/description/emma_core.xacro (robot description, xacro)
@@ -13,6 +13,28 @@
     <link name="base_link">
     </link>
+    <!-- Chassis Link or Main Body -->
+    <link name="chassis">
+    <visual>
+        <!-- <origin rpy="0 0 0" xyz="0 0 0"/> -->
+        <origin rpy="1.5707963267949 0 1.5707963267949" xyz="0 0 0"/>
+        <geometry>
+        <!-- <box size="0.4 0.3 0.1"/> -->
+         <mesh filename="file:///home/osama/schaeffler/src/emma_visualization/meshes/AMR_Platform.STL"/>
+        </geometry>
+        <material name="Gazebo/Red"/>
+    </visual>
+    <collision>
+        <origin rpy="0 0 0" xyz="0 0 0"/>
+        <geometry>
+        <box size="0.4 0.3 0.1"/>
+        </geometry>
+    </collision>
+    <inertial>
+        <mass value="4.07"/>
+        <inertia ixx="0.426" ixy="0.0" ixz="0.0" iyy="0.496" iyz="0.0" izz="0.91"/>
+    </inertial>
+    </link>
     <!-- Chassis Link or Main Body-->
-    <link name="chassis">
+    <!-- <link name="chassis">
         <visual>
             <origin rpy="1.5707963267949 0 1.5707963267949" xyz="0 0 0"/>
@@ -32,5 +54,9 @@
             <inertia ixx="0.426" ixy="0.0" ixz="0.0" iyy="0.496" iyz="0.0" izz="0.91"/>
         </inertial>
-    </link>
+    </link> -->
+<!--
+    <gazebo reference="chassis">
+        <material>Gazebo/white</material>
+    </gazebo> -->
     <!-- Chassis Joint-->
     <joint name="chassis_joint" type="fixed">
@@ -64,5 +90,5 @@
             <axis xyz="0 1 0"/>
     </joint>
-    <gazebo reference="chassis">
+    <gazebo reference="left_wheel">
         <material>Gazebo/black</material>
     </gazebo>
@@ -92,5 +118,5 @@
             <axis xyz="0 1 0"/>
     </joint>
-    <gazebo reference="chassis">
+    <gazebo reference="right_wheel">
         <material>Gazebo/black</material>
     </gazebo>
@@ -120,5 +146,5 @@
         <origin xyz="0.209 -0.108 -0.049" rpy="0 0 0"/>
     </joint>
-    <gazebo reference="chassis">
+    <gazebo reference="right_front_small_wheel">
         <material>Gazebo/black</material>
     </gazebo>
@@ -148,5 +174,5 @@
         <origin  xyz="0.209 0.108 -0.049" rpy="0 0 0"/>
     </joint>
-    <gazebo reference="chassis">
+    <gazebo reference="left_front_small_wheel">
         <material>Gazebo/black</material>
     </gazebo>
@@ -176,5 +202,5 @@
         <origin xyz="-0.228 0.156 -0.049" rpy="0 0 0" />
     </joint>
-     <gazebo reference="chassis">
+     <gazebo reference="left_back_small_wheel">
         <material>Gazebo/black</material>
     </gazebo>
@@ -204,5 +230,5 @@
         <origin xyz="-0.228 -0.156 -0.049" rpy="0 0 0" />
     </joint>
-    <gazebo reference="chassis">
+    <gazebo reference="right_back_small_wheel">
         <material>Gazebo/black</material>
     </gazebo>
