Commit message: lidar adjustments

File: src/emma_visualization/description/lidar.xacro (robot description, xacro)
@@ -4,5 +4,5 @@
         <parent link="chassis"/>
         <child link="laser_frame"/>
-        <origin xyz="1 0 2" rpy="0 0 0"/>
+        <origin xyz="0.3 0 0.11" rpy="0 0 0"/>
     </joint>
     <link name="laser_frame">
@@ -35,6 +35,6 @@
                     <horizontal>
                         <samples>360</samples>
-                        <min_angle>-3.14</min_angle>
-                        <max_angle>3.14</max_angle>
+                        <min_angle>-1.570796</min_angle>
+                        <max_angle>1.570796</max_angle>
                     </horizontal>
                 </scan>

Commit message: .

File: src/emma_visualization/description/lidar.xacro (robot description, xacro)
@@ -11,5 +11,5 @@
                 <cylinder radius="0.05" length="0.04"/>
             </geometry>
-            <!-- <material name="red"/> -->
+            <material name="red"/>
         </visual>
         <collision>
