Commit message: STL added and loaded

File: src/emma_visualization/description/emma_core.xacro (robot description, xacro)
@@ -24,6 +24,5 @@
             <origin rpy="1.5707963267949 0 1.5707963267949" xyz="0 0 0"/>
             <geometry>
-                <!-- <mesh filename="package://amr_visualisation/meshes/AMR_Platform.STL"/> -->
-                <box size="0.4 0.2 0.5"/>
+                <mesh filename="package://emma_visualization/meshes/emma_cover.stl"/>
             </geometry>
             <material name="white"/>
@@ -32,6 +31,5 @@
             <origin rpy="1.5707963267949 0 1.5707963267949" xyz="0 0 0"/>
             <geometry>
-                <!-- <mesh filename="package://amr_visualisation/meshes/AMR_Platform.STL"/> -->
-                <box size="0.4 0.2 0.5"/>
+                <mesh filename="package://emma_visualization/meshes/emma_cover.stl"/>
             </geometry>
         </collision>

Commit message: left and right wheels added

File: src/emma_visualization/description/emma_core.xacro (robot description, xacro)
@@ -10,14 +10,8 @@
         <color rgba="1 1 1 1"/>
     </material>
+    <!-- Base Link-->
     <link name="base_link">
     </link>
-    <!-- <link name="chassis">
-        <visual>
-            <origin xyz="0.0 0.0 0.0" rpy="0.0 0.0 0.0"/>
-            <geometry>
-                <box size="0.4 0.2 0.5"/>
-            </geometry>
-        </visual>
-    </link> -->
+    <!-- Chassis Link or Main Body-->
     <link name="chassis">
         <visual>
@@ -37,10 +31,89 @@
             <mass value="4.07"/>
             <inertia ixx="0.426" ixy="0.0" ixz="0.0" iyy="0.496" iyz="0.0" izz="0.91"/>
-            </inertial>
+        </inertial>
     </link>
+    <!-- Chassis Joint-->
     <joint name="chassis_joint" type="fixed">
         <parent link="base_link"/>
         <child link="chassis"/>
-        <origin xyz="0.0 0.0 0.1"/>
+        <origin xyz="0.0 0.0 0.085"/>
     </joint>
+    <link name="left_wheel">
+        <visual>
+        <origin xyz="0 0 0" rpy="1.5707963267949 0 0" />
+        <geometry>
+            <cylinder radius="0.088" length="0.03937"/>
+        </geometry>
+        <material name="black"/>
+        </visual>
+        <collision>
+        <origin xyz="0 0 0" rpy="1.5707963267949 0 0"/>
+        <geometry>
+            <cylinder radius="0.088" length="0.03937"/>
+        </geometry>
+        </collision>
+        <inertial>
+        <mass value="0.17"/>
+        <inertia ixx="0.000204" ixy="0.0" ixz="0.0" iyy="0.000306" iyz="0.0" izz="0.000204"/>
+        </inertial>
+    </link>
+    <joint name="left_wheel_joint" type="continuous">
+            <parent link="chassis"/>
+            <child link="left_wheel"/>
+            <origin xyz="0 0.196425 0.000881" rpy="0 0 0"/>
+            <axis xyz="0 1 0"/>
+    </joint>
+    <link name="right_wheel">
+        <visual>
+        <origin xyz="0 0 0" rpy="1.5707963267949 0 0" />
+        <geometry>
+            <cylinder radius="0.088" length="0.03937"/>
+        </geometry>
+        <material name="black"/>
+        </visual>
+        <collision>
+        <origin xyz="0 0 0" rpy="1.5707963267949 0 0"/>
+        <geometry>
+            <cylinder radius="0.088" length="0.03937"/>
+        </geometry>
+        </collision>
+        <inertial>
+        <mass value="0.17"/>
+        <inertia ixx="0.000204" ixy="0.0" ixz="0.0" iyy="0.000306" iyz="0.0" izz="0.000204"/>
+        </inertial>
+    </link>
+    <joint name="right_wheel_joint" type="continuous">
+            <parent link="chassis"/>
+            <child link="right_wheel"/>
+            <origin xyz="0 -0.196425 0.000881" rpy="0 0 0"/>
+            <axis xyz="0 1 0"/>
+    </joint>
+    <!-- <link name="left_wheel">
+    <visual>
+        <geometry>
+            <cylinder radius="0.088" length="0.03937"/>
+        </geometry>
+        <material name="blue"/>
+    </visual>
+    </link>
+    <joint name="left_wheel_joint" type="continuous">
+        <parent link="chassis"/>
+        <child link="left_wheel"/>
+        <origin xyz="0.0 0.6 0.0" rpy="-${pi/2} 0 0"/>
+        <axis xyz="0.0 0.0 1.0"/>
+    </joint>
+    <link name="right_wheel">
+    <visual>
+        <geometry>
+            <cylinder radius="0.05" length="0.04"/>
+        </geometry>
+        <material name="blue"/>
+    </visual>
+    </link>
+    <joint name="right_wheel_joint" type="continuous">
+        <parent link="base_link"/>
+        <child link="right_wheel"/>
+        <origin xyz="0.0 -0.6 0.0" rpy="${pi/2} 0 0"/>
+        <axis xyz="0.0 0.0 -1.0"/>
+    </joint> -->
 </robot>

Commit message: left and right  front wheels

File: src/emma_visualization/description/emma_core.xacro (robot description, xacro)
@@ -89,4 +89,54 @@
             <axis xyz="0 1 0"/>
     </joint>
+    <link name="right_front_small_wheel">
+        <visual>
+            <origin xyz="0 0 0" rpy="1.5707963267949 0 0"/>
+            <geometry>
+                <cylinder length="0.02775" radius="0.0375"/>
+            </geometry>
+            <material name="black"/>
+        </visual>
+        <collision>
+            <origin xyz="0 0 0" rpy="1.5707963267949 0 0"/>
+            <geometry>
+                <cylinder length="0.02775" radius="0.0375"/>
+            </geometry>
+        </collision>
+        <inertial>
+            <mass value="0.17"/>
+            <inertia ixx="0.000204" ixy="0.0" ixz="0.0" iyy="0.000306" iyz="0.0" izz="0.000204"/>
+        </inertial>
+    </link>
+    <joint name="right_front_small_wheel_joint" type="continuous">
+        <axis rpy="0 0 0" xyz="0 1 0"/>
+        <parent link="chassis"/>
+        <child link="right_front_small_wheel"/>
+        <origin rpy="3.1415926535897 0 0" xyz="0.209 -0.108 -0.049"/>
+    </joint>
+    <link name="left_front_small_wheel">
+        <visual>
+            <origin xyz="0 0 0" rpy="1.5707963267949 0 0"/>
+            <geometry>
+                <cylinder length="0.02775" radius="0.0375"/>
+            </geometry>
+            <material name="black"/>
+        </visual>
+        <collision>
+            <origin xyz="0 0 0" rpy="1.5707963267949 0 0"/>
+            <geometry>
+                <cylinder length="0.02775" radius="0.0375"/>
+            </geometry>
+        </collision>
+        <inertial>
+            <mass value="0.17"/>
+            <inertia ixx="0.000204" ixy="0.0" ixz="0.0" iyy="0.000306" iyz="0.0" izz="0.000204"/>
+        </inertial>
+    </link>
+    <joint name="left_front_small_wheel_joint" type="continuous">
+        <axis rpy="0 0 0" xyz="0 1 0"/>
+        <parent link="chassis"/>
+        <child link="left_front_small_wheel"/>
+        <origin rpy="3.1415926535897 0 0" xyz="0.209 0.108 -0.049"/>
+    </joint>
     <!-- <link name="left_wheel">
     <visual>

Commit message: Maintain consistency

File: src/emma_visualization/description/emma_core.xacro (robot description, xacro)
@@ -112,5 +112,5 @@
         <parent link="chassis"/>
         <child link="right_front_small_wheel"/>
-        <origin rpy="3.1415926535897 0 0" xyz="0.209 -0.108 -0.049"/>
+        <origin xyz="0.209 -0.108 -0.049" rpy="3.1415926535897 0 0"/>
     </joint>
     <link name="left_front_small_wheel">
@@ -137,5 +137,5 @@
         <parent link="chassis"/>
         <child link="left_front_small_wheel"/>
-        <origin rpy="3.1415926535897 0 0" xyz="0.209 0.108 -0.049"/>
+        <origin  xyz="0.209 0.108 -0.049" rpy="3.1415926535897 0 0"/>
     </joint>
     <!-- <link name="left_wheel">

Commit message: Left and right back wheels

File: src/emma_visualization/description/emma_core.xacro (robot description, xacro)
@@ -139,4 +139,54 @@
         <origin  xyz="0.209 0.108 -0.049" rpy="3.1415926535897 0 0"/>
     </joint>
+    <link name="left_back_small_wheel">
+        <visual>
+            <origin xyz="0 0 0" rpy="1.5707963267949 0 0" />
+            <geometry>
+                <cylinder length="0.02775" radius="0.0375"/>
+            </geometry>
+            <material name="black"/>
+        </visual>
+        <collision>
+            <origin xyz="0 0 0" rpy="1.5707963267949 0 0" />
+            <geometry>
+                <cylinder length="0.02775" radius="0.0375"/>
+            </geometry>
+        </collision>
+        <inertial>
+            <mass value="0.17"/>
+            <inertia ixx="0.000204" ixy="0.0" ixz="0.0" iyy="0.000306" iyz="0.0" izz="0.000204"/>
+        </inertial>
+    </link>
+    <joint name="left_back_small_wheel_joint" type="continuous">
+        <axis rpy="0 0 0" xyz="0 1 0"/>
+        <parent link="chassis"/>
+        <child link="left_back_small_wheel"/>
+        <origin xyz="-0.228 0.156 -0.049" rpy="0 0 0" />
+    </joint>
+    <link name="right_back_small_wheel">
+        <visual>
+            <origin xyz="0 0 0" rpy="1.5707963267949 0 0" />
+            <geometry>
+                <cylinder length="0.02775" radius="0.0375"/>
+            </geometry>
+            <material name="black"/>
+        </visual>
+        <collision>
+            <origin xyz="0 0 0" rpy="1.5707963267949 0 0" />
+            <geometry>
+                <cylinder length="0.02775" radius="0.0375"/>
+            </geometry>
+        </collision>
+        <inertial>
+            <mass value="0.17"/>
+            <inertia ixx="0.000204" ixy="0.0" ixz="0.0" iyy="0.000306" iyz="0.0" izz="0.000204"/>
+        </inertial>
+    </link>
+    <joint name="right_back_small_wheel_joint" type="continuous">
+        <axis rpy="0 0 0" xyz="0 1 0"/>
+        <parent link="chassis"/>
+        <child link="right_back_small_wheel"/>
+        <origin xyz="-0.228 -0.156 -0.049" rpy="0 0 0" />
+    </joint>
     <!-- <link name="left_wheel">
     <visual>

Commit message: Orientation corrected

File: src/emma_visualization/description/emma_core.xacro (robot description, xacro)
@@ -112,5 +112,5 @@
         <parent link="chassis"/>
         <child link="right_front_small_wheel"/>
-        <origin xyz="0.209 -0.108 -0.049" rpy="3.1415926535897 0 0"/>
+        <origin xyz="0.209 -0.108 -0.049" rpy="0 0 0"/>
     </joint>
     <link name="left_front_small_wheel">
@@ -137,5 +137,5 @@
         <parent link="chassis"/>
         <child link="left_front_small_wheel"/>
-        <origin  xyz="0.209 0.108 -0.049" rpy="3.1415926535897 0 0"/>
+        <origin  xyz="0.209 0.108 -0.049" rpy="0 0 0"/>
     </joint>
     <link name="left_back_small_wheel">

Commit message: changes loading STL with absoluate path

File: src/emma_visualization/description/emma_core.xacro (robot description, xacro)
@@ -18,5 +18,5 @@
             <origin rpy="1.5707963267949 0 1.5707963267949" xyz="0 0 0"/>
             <geometry>
-                <mesh filename="package://emma_visualization/meshes/emma_cover.stl"/>
+                <mesh filename="file:///home/osama/schaeffler/src/emma_visualization/meshes/AMR_Platform.STL"/>
             </geometry>
             <material name="white"/>
@@ -25,5 +25,5 @@
             <origin rpy="1.5707963267949 0 1.5707963267949" xyz="0 0 0"/>
             <geometry>
-                <mesh filename="package://emma_visualization/meshes/emma_cover.stl"/>
+                <mesh filename="file:///home/osama/schaeffler/src/emma_visualization/meshes/AMR_Platform.STL"/>
             </geometry>
         </collision>
@@ -64,4 +64,7 @@
             <axis xyz="0 1 0"/>
     </joint>
+    <gazebo reference="chassis">
+        <material>Gazebo/black</material>
+    </gazebo>
     <link name="right_wheel">
         <visual>
@@ -89,4 +92,7 @@
             <axis xyz="0 1 0"/>
     </joint>
+    <gazebo reference="chassis">
+        <material>Gazebo/black</material>
+    </gazebo>
     <link name="right_front_small_wheel">
         <visual>
@@ -114,4 +120,7 @@
         <origin xyz="0.209 -0.108 -0.049" rpy="0 0 0"/>
     </joint>
+    <gazebo reference="chassis">
+        <material>Gazebo/black</material>
+    </gazebo>
     <link name="left_front_small_wheel">
         <visual>
@@ -139,4 +148,7 @@
         <origin  xyz="0.209 0.108 -0.049" rpy="0 0 0"/>
     </joint>
+    <gazebo reference="chassis">
+        <material>Gazebo/black</material>
+    </gazebo>
     <link name="left_back_small_wheel">
         <visual>
@@ -164,4 +176,7 @@
         <origin xyz="-0.228 0.156 -0.049" rpy="0 0 0" />
     </joint>
+     <gazebo reference="chassis">
+        <material>Gazebo/black</material>
+    </gazebo>
     <link name="right_back_small_wheel">
         <visual>
@@ -189,4 +204,7 @@
         <origin xyz="-0.228 -0.156 -0.049" rpy="0 0 0" />
     </joint>
+    <gazebo reference="chassis">
+        <material>Gazebo/black</material>
+    </gazebo>
     <!-- <link name="left_wheel">
     <visual>

Commit message: color correction

File: src/emma_visualization/description/emma_core.xacro (robot description, xacro)
@@ -20,7 +20,7 @@
         <geometry>
         <!-- <box size="0.4 0.3 0.1"/> -->
-         <mesh filename="file:///home/osama/schaeffler/src/emma_visualization/meshes/AMR_Platform.STL"/>
-        </geometry>
-        <material name="Gazebo/Red"/>
+         <mesh filename="file:///home/schaeffler/schaeffler/src/emma_visualization/meshes/AMR_Platform.STL"/>
+        </geometry>
+        <material name="white"/>
     </visual>
     <collision>
@@ -65,4 +65,7 @@
         <origin xyz="0.0 0.0 0.085"/>
     </joint>
+    <gazebo reference="chassis">
+        <material>Gazebo/white</material>
+    </gazebo>
     <link name="left_wheel">
         <visual>

Commit message: arranged tags

File: src/emma_visualization/description/emma_core.xacro (robot description, xacro)
@@ -35,4 +35,13 @@
     </inertial>
     </link>
+    <!-- Chassis Joint-->
+    <joint name="chassis_joint" type="fixed">
+        <parent link="base_link"/>
+        <child link="chassis"/>
+        <origin xyz="0.0 0.0 0.085"/>
+    </joint>
+    <gazebo reference="chassis">
+        <material>Gazebo/white</material>
+    </gazebo>
     <!-- Chassis Link or Main Body-->
     <!-- <link name="chassis">
@@ -59,30 +68,21 @@
         <material>Gazebo/white</material>
     </gazebo> -->
-    <!-- Chassis Joint-->
-    <joint name="chassis_joint" type="fixed">
-        <parent link="base_link"/>
-        <child link="chassis"/>
-        <origin xyz="0.0 0.0 0.085"/>
-    </joint>
-    <gazebo reference="chassis">
-        <material>Gazebo/white</material>
-    </gazebo>
     <link name="left_wheel">
         <visual>
-        <origin xyz="0 0 0" rpy="1.5707963267949 0 0" />
-        <geometry>
-            <cylinder radius="0.088" length="0.03937"/>
-        </geometry>
-        <material name="black"/>
-        </visual>
-        <collision>
-        <origin xyz="0 0 0" rpy="1.5707963267949 0 0"/>
-        <geometry>
-            <cylinder radius="0.088" length="0.03937"/>
-        </geometry>
-        </collision>
-        <inertial>
-        <mass value="0.17"/>
-        <inertia ixx="0.000204" ixy="0.0" ixz="0.0" iyy="0.000306" iyz="0.0" izz="0.000204"/>
+            <origin xyz="0 0 0" rpy="1.5707963267949 0 0" />
+            <geometry>
+                <cylinder radius="0.088" length="0.03937"/>
+            </geometry>
+            <material name="black"/>
+        </visual>
+        <collision>
+            <origin xyz="0 0 0" rpy="1.5707963267949 0 0"/>
+            <geometry>
+                <cylinder radius="0.088" length="0.03937"/>
+            </geometry>
+        </collision>
+        <inertial>
+            <mass value="0.17"/>
+            <inertia ixx="0.000204" ixy="0.0" ixz="0.0" iyy="0.000306" iyz="0.0" izz="0.000204"/>
         </inertial>
     </link>
@@ -98,19 +98,19 @@
     <link name="right_wheel">
         <visual>
-        <origin xyz="0 0 0" rpy="1.5707963267949 0 0" />
-        <geometry>
-            <cylinder radius="0.088" length="0.03937"/>
-        </geometry>
-        <material name="black"/>
-        </visual>
-        <collision>
-        <origin xyz="0 0 0" rpy="1.5707963267949 0 0"/>
-        <geometry>
-            <cylinder radius="0.088" length="0.03937"/>
-        </geometry>
-        </collision>
-        <inertial>
-        <mass value="0.17"/>
-        <inertia ixx="0.000204" ixy="0.0" ixz="0.0" iyy="0.000306" iyz="0.0" izz="0.000204"/>
+            <origin xyz="0 0 0" rpy="1.5707963267949 0 0" />
+            <geometry>
+                <cylinder radius="0.088" length="0.03937"/>
+            </geometry>
+            <material name="black"/>
+        </visual>
+        <collision>
+            <origin xyz="0 0 0" rpy="1.5707963267949 0 0"/>
+            <geometry>
+                <cylinder radius="0.088" length="0.03937"/>
+            </geometry>
+        </collision>
+        <inertial>
+            <mass value="0.17"/>
+            <inertia ixx="0.000204" ixy="0.0" ixz="0.0" iyy="0.000306" iyz="0.0" izz="0.000204"/>
         </inertial>
     </link>
@@ -236,31 +236,3 @@
         <material>Gazebo/black</material>
     </gazebo>
-    <!-- <link name="left_wheel">
-    <visual>
-        <geometry>
-            <cylinder radius="0.088" length="0.03937"/>
-        </geometry>
-        <material name="blue"/>
-    </visual>
-    </link>
-    <joint name="left_wheel_joint" type="continuous">
-        <parent link="chassis"/>
-        <child link="left_wheel"/>
-        <origin xyz="0.0 0.6 0.0" rpy="-${pi/2} 0 0"/>
-        <axis xyz="0.0 0.0 1.0"/>
-    </joint>
-    <link name="right_wheel">
-    <visual>
-        <geometry>
-            <cylinder radius="0.05" length="0.04"/>
-        </geometry>
-        <material name="blue"/>
-    </visual>
-    </link>
-    <joint name="right_wheel_joint" type="continuous">
-        <parent link="base_link"/>
-        <child link="right_wheel"/>
-        <origin xyz="0.0 -0.6 0.0" rpy="${pi/2} 0 0"/>
-        <axis xyz="0.0 0.0 -1.0"/>
-    </joint> -->
 </robot>

Commit message: arranged

File: src/emma_visualization/description/emma_core.xacro (robot description, xacro)
@@ -35,4 +35,7 @@
     </inertial>
     </link>
+    <gazebo reference="chassis">
+        <material>Gazebo/white</material>
+    </gazebo>
     <!-- Chassis Joint-->
     <joint name="chassis_joint" type="fixed">
@@ -41,7 +44,4 @@
         <origin xyz="0.0 0.0 0.085"/>
     </joint>
-    <gazebo reference="chassis">
-        <material>Gazebo/white</material>
-    </gazebo>
     <!-- Chassis Link or Main Body-->
     <!-- <link name="chassis">
@@ -87,4 +87,7 @@
         </inertial>
     </link>
+    <gazebo reference="left_wheel">
+        <material>Gazebo/black</material>
+    </gazebo>
     <joint name="left_wheel_joint" type="continuous">
             <parent link="chassis"/>
@@ -93,7 +96,4 @@
             <axis xyz="0 1 0"/>
     </joint>
-    <gazebo reference="left_wheel">
-        <material>Gazebo/black</material>
-    </gazebo>
     <link name="right_wheel">
         <visual>
@@ -115,4 +115,7 @@
         </inertial>
     </link>
+    <gazebo reference="right_wheel">
+        <material>Gazebo/black</material>
+    </gazebo>
     <joint name="right_wheel_joint" type="continuous">
             <parent link="chassis"/>
@@ -121,7 +124,4 @@
             <axis xyz="0 1 0"/>
     </joint>
-    <gazebo reference="right_wheel">
-        <material>Gazebo/black</material>
-    </gazebo>
     <link name="right_front_small_wheel">
         <visual>
@@ -143,4 +143,7 @@
         </inertial>
     </link>
+    <gazebo reference="right_front_small_wheel">
+        <material>Gazebo/black</material>
+    </gazebo>
     <joint name="right_front_small_wheel_joint" type="continuous">
         <axis rpy="0 0 0" xyz="0 1 0"/>
@@ -149,7 +152,4 @@
         <origin xyz="0.209 -0.108 -0.049" rpy="0 0 0"/>
     </joint>
-    <gazebo reference="right_front_small_wheel">
-        <material>Gazebo/black</material>
-    </gazebo>
     <link name="left_front_small_wheel">
         <visual>
@@ -171,4 +171,7 @@
         </inertial>
     </link>
+    <gazebo reference="left_front_small_wheel">
+        <material>Gazebo/black</material>
+    </gazebo>
     <joint name="left_front_small_wheel_joint" type="continuous">
         <axis rpy="0 0 0" xyz="0 1 0"/>
@@ -177,7 +180,4 @@
         <origin  xyz="0.209 0.108 -0.049" rpy="0 0 0"/>
     </joint>
-    <gazebo reference="left_front_small_wheel">
-        <material>Gazebo/black</material>
-    </gazebo>
     <link name="left_back_small_wheel">
         <visual>
@@ -199,4 +199,7 @@
         </inertial>
     </link>
+     <gazebo reference="left_back_small_wheel">
+        <material>Gazebo/black</material>
+    </gazebo>
     <joint name="left_back_small_wheel_joint" type="continuous">
         <axis rpy="0 0 0" xyz="0 1 0"/>
@@ -205,7 +208,4 @@
         <origin xyz="-0.228 0.156 -0.049" rpy="0 0 0" />
     </joint>
-     <gazebo reference="left_back_small_wheel">
-        <material>Gazebo/black</material>
-    </gazebo>
     <link name="right_back_small_wheel">
         <visual>
@@ -227,4 +227,7 @@
         </inertial>
     </link>
+    <gazebo reference="right_back_small_wheel">
+        <material>Gazebo/black</material>
+    </gazebo>
     <joint name="right_back_small_wheel_joint" type="continuous">
         <axis rpy="0 0 0" xyz="0 1 0"/>
@@ -233,6 +236,3 @@
         <origin xyz="-0.228 -0.156 -0.049" rpy="0 0 0" />
     </joint>
-    <gazebo reference="right_back_small_wheel">
-        <material>Gazebo/black</material>
-    </gazebo>
 </robot>

Commit message: changed wheel type to fixed

File: src/emma_visualization/description/emma_core.xacro (robot description, xacro)
@@ -146,5 +146,5 @@
         <material>Gazebo/black</material>
     </gazebo>
-    <joint name="right_front_small_wheel_joint" type="continuous">
+    <joint name="right_front_small_wheel_joint" type="fixed">
         <axis rpy="0 0 0" xyz="0 1 0"/>
         <parent link="chassis"/>
@@ -174,5 +174,5 @@
         <material>Gazebo/black</material>
     </gazebo>
-    <joint name="left_front_small_wheel_joint" type="continuous">
+    <joint name="left_front_small_wheel_joint" type="fixed">
         <axis rpy="0 0 0" xyz="0 1 0"/>
         <parent link="chassis"/>
@@ -202,5 +202,5 @@
         <material>Gazebo/black</material>
     </gazebo>
-    <joint name="left_back_small_wheel_joint" type="continuous">
+    <joint name="left_back_small_wheel_joint" type="fixed">
         <axis rpy="0 0 0" xyz="0 1 0"/>
         <parent link="chassis"/>
@@ -230,5 +230,5 @@
         <material>Gazebo/black</material>
     </gazebo>
-    <joint name="right_back_small_wheel_joint" type="continuous">
+    <joint name="right_back_small_wheel_joint" type="fixed">
         <axis rpy="0 0 0" xyz="0 1 0"/>
         <parent link="chassis"/>

Commit message: collision adjustment

File: src/emma_visualization/description/emma_core.xacro (robot description, xacro)
@@ -25,7 +25,7 @@
     </visual>
     <collision>
-        <origin rpy="0 0 0" xyz="0 0 0"/>
+        <origin rpy="0 0 0" xyz="0 0 0.05"/>
         <geometry>
-        <box size="0.4 0.3 0.1"/>
+        <box size="0.4 0.3 0.2"/>
         </geometry>
     </collision>
