Commit message: stashed

File: src/emma_visualization/description/emma_core.xacro (robot description, xacro)
@@ -20,5 +20,6 @@
         <geometry>
         <!-- <box size="0.4 0.3 0.1"/> -->
-         <mesh filename="file:///home/schaeffler/schaeffler/src/emma_visualization/meshes/AMR_Platform.STL"/>
+         <!-- <mesh filename="file:///home/osama/schaeffler/src/emma_visualization/meshes/AMR_Platform.STL"/> -->
+            <mesh filename="file:///home/osama/schaeffler/src/emma_visualization/meshes/AMR_Platform.STL"/>
         </geometry>
         <material name="white"/>

Commit message: red color added

File: src/emma_visualization/description/emma_core.xacro (robot description, xacro)
@@ -9,4 +9,7 @@
     <material name="white">
         <color rgba="1 1 1 1"/>
+    </material>
+    <material name="red">
+        <color rgba="1 0 0 1"/>
     </material>
     <!-- Base Link-->

Commit message: footprint as parent of baselink

File: src/emma_visualization/description/emma_core.xacro (robot description, xacro)
@@ -15,4 +15,12 @@
     <!-- Base Link-->
     <link name="base_link">
+    </link>
+    <!-- BASE_FOOTPRINT LINK -->
+    <joint name="base_footprint_joint" type="fixed">
+        <parent link="base_link"/>
+        <child link="base_footprint"/>
+        <origin xyz="0 0 0" rpy="0 0 0"/>
+    </joint>
+    <link name="base_footprint">
     </link>
     <!-- Chassis Link or Main Body -->
@@ -23,6 +31,6 @@
         <geometry>
         <!-- <box size="0.4 0.3 0.1"/> -->
-         <!-- <mesh filename="file:///home/osama/schaeffler/src/emma_visualization/meshes/AMR_Platform.STL"/> -->
-            <mesh filename="file:///home/osama/schaeffler/src/emma_visualization/meshes/AMR_Platform.STL"/>
+         <mesh filename="file:///home/schaeffler/schaeffler/src/emma_visualization/meshes/AMR_Platform.STL"/>
+            <!-- <mesh filename="file:///home/osama/schaeffler/src/emma_visualization/meshes/AMR_Platform.STL"/> -->
         </geometry>
         <material name="white"/>
